Commit message: Add files via upload

File: cartographer_ros/urdf/kit_2d.urdf (robot description, URDF)
Before this commit: robot cartographer_backpack_3d, 3 links, 2 joints
Joints:
- joint velo_link_joint: origin xyz=0.81 0.32 0.8 rpy=0.0 0.0 0.0 -> xyz=-0.80 0.31 -0.79 rpy=0.0148239 -0.0010179 -0.0007629; parent base_link -> imu_link
